File: Design/H01R01.brd (EAGLE design)
At the start: 34.6 x 30 mm, 31 parts, among them P1 HEXABIT_17.32, Q1 MMBT3904LT1, Q2 MMBT3904LT1, Q3 MMBT3904LT1, X1 XTALL_CSTCE8M00G52

Commit message: first edit
Parts:
- removed D2: CREE-CLVBA-FKA-CC1F1L1BB7R3R3, Hexabitz:PCB-1023943-1
- removed Q1, Q2, Q3: MMBT3904LT1, Hexabitz:MMBT3904LT1
- removed R4: 68.0R, Hexabitz:R-0603
- removed R5, R6: 10.0R, Hexabitz:R-0603
- removed R7, R8, R9: 2400.0R, Hexabitz:R-0603
- added C10: 100nF, HEXABITZ_RCLS:C-0603
- added R57, R58: 4.7k, HEXABITZ_RCLS:R-0603
- added U2: TSD305-1C55, HEXABITZ_ICs:TEMPERATURESENSOR-TO5
Connections:
- removed net N$1: D2.P$1, R4.1
- removed net N$10: Q1.3, R6.2
- removed net N$11: Q2.3, R5.2
- removed net N$12: Q3.3, R4.2
- removed net N$13: Q1.1, R7.2
- removed net N$14: Q2.1, R8.2
- removed net N$15: Q3.1, R9.2
- removed net N$2: D2.P$4, R5.1
- removed net N$8: D2.P$3, R6.1
- new net +3V3: C10.1, R57.2, R58.2, U2.3
- new net I2C_SCL_IR_2: R57.1, U2.1
- new net I2C_SDA_IR_2: R58.1, U2.2
- net BLED: no longer R7.1
- net GLED: no longer R8.1
- net GND: now also C10.2, U2.4; no longer Q1.2, Q2.2, Q3.2
- net RLED: no longer R9.1
- net VDD: no longer D2.P$2
Routing:
- net GND: track 153.1 -> 137.7 mm
- net N$12: track 6.09 -> 0.00 mm
- net N$2: track 3.42 -> 0.00 mm
- net N$15: track 3.22 -> 0.00 mm
- net N$11: track 3.08 -> 0.00 mm
- net N$8: track 3.03 -> 0.00 mm
- net N$1: track 2.63 -> 0.00 mm
- net N$13: track 1.94 -> 0.00 mm
- net N$14: track 1.92 -> 0.00 mm
- net N$10: track 1.90 -> 0.00 mm
- net GLED: track 10.3 -> 9.36 mm
- net VDD: track 136.5 -> 135.7 mm
