File: Design/H01R01.sch (EAGLE design)
At the start: 31 parts, among them P1 HEXABIT_17.32, Q1 MMBT3904LT1, Q2 MMBT3904LT1, Q3 MMBT3904LT1, X1 XTALL_CSTCE8M00G52

Commit message: first edit
Parts:
- removed D2: CREE-CLVBA-FKA-CC1F1L1BB7R3R3, Hexabitz:CREE-CLVBA-FKA-CC1F1L1BB7R3R3
- removed Q1, Q2, Q3: MMBT3904LT1, Hexabitz:MMBT3904LT1
- removed R4: 68.0R, Hexabitz:R-0603
- removed R5, R6: 10.0R, Hexabitz:R-0603
- removed R7, R8, R9: 2400.0R, Hexabitz:R-0603
- added C10: 100nF, HEXABITZ_RCLS:C-0603
- added R57, R58: 4.7k, HEXABITZ_RCLS:R-0603
- added U2: TSD305-1C55, HEXABITZ_ICs:TSD305-1C55
Connections:
- removed net N$1: D2.CRED, R4.1
- removed net N$10: Q1.C, R6.2
- removed net N$11: Q2.C, R5.2
- removed net N$12: Q3.C, R4.2
- removed net N$13: Q1.B, R7.2
- removed net N$14: Q2.B, R8.2
- removed net N$15: Q3.B, R9.2
- removed net N$2: D2.CGREEN, R5.1
- removed net N$8: D2.CBLUE, R6.1
- new net +3V3: C10.1, R57.2, R58.2, U2.VDD
- new net I2C_SCL_IR_2: R57.1, U2.SCL
- new net I2C_SDA_IR_2: R58.1, U2.SDA
- net BLED: no longer R7.1
- net GLED: no longer R8.1
- net GND: now also C10.2, U2.GND; no longer Q1.E, Q2.E, Q3.E
- net RLED: no longer R9.1
- net VDD: no longer D2.A2
Other:
- note added: "H09R9"
- note added: "H09R9_Frontend"
- note added: "I2C Bus 2"
- note added: "IR termpratuer sensor _ Digital I2C comunication"
- note added: "Thermopile Sensor"
- note removed: "H01R0"
- note removed: "RGB LED"
