File: Design/H09R9x.brd (EAGLE design)
At the start: 34.6 x 30 mm, 24 parts, among them P1 HEXABIT_17.32, U1 STM32F091CBU6, U2 TSD305-1C55, X1 XTALL_CSTCE8M00G52

Commit message: brd edit
Parts:
- moved D1 9.40 mm to (25.4, 42.3)
- moved R1 7.30 mm to (27.8, 42.2)
- moved B 6.59 mm to (37.3, 47.4)
- moved C1 4.49 mm to (44.9, 33.2)
- moved R 2.65 mm to (47.3, 38.4), turned to 180 degrees
- moved C 2.17 mm to (24.8, 38.0)
- moved R2 1.70 mm to (40.0, 47.0), turned to 180 degrees
- moved D 1.48 mm to (27.4, 38.0)
- moved C5 1.42 mm to (41.4, 36.2)
- moved C2 1.30 mm to (43.4, 36.1)
- moved FB1 1.05 mm to (44.1, 30.9)
- moved R3 1.05 mm to (45.4, 36.3)
- moved C7 1.02 mm to (28.9, 43.6)
- moved X1 0.76 mm to (41.2, 40.6)
- moved C4 0.40 mm to (26.8, 43.1)
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Routing:
- net I2C2_SCL: track 0.00 -> 27.6 mm, vias 0 -> 1
- net I2C2_SDA: track 0.00 -> 26.3 mm, vias 0 -> 1
- net USART6_TX: track 0.00 -> 20.6 mm, vias 0 -> 1
- net USART6_RX: track 0.00 -> 19.4 mm
- net USART4_RX: track 0.00 -> 18.9 mm, vias 0 -> 2
- net USART4_TX: track 0.00 -> 17.3 mm, vias 0 -> 1
- net USART1_TX: track 0.00 -> 16.5 mm, vias 0 -> 1
- net USART2_RX: track 0.00 -> 16.4 mm
- net USART2_TX: track 0.00 -> 15.9 mm, vias 0 -> 1
- net USART1_RX: track 0.00 -> 15.5 mm
- net VDDA: track 0.00 -> 13.8 mm, vias 0 -> 1
- net VDD: track 14.2 -> 27.7 mm, vias 0 -> 3
- net R1: track 7.88 -> 18.5 mm
- net GND: track 13.8 -> 21.0 mm, vias 2 -> 5
- net N$3: track 0.00 -> 4.71 mm, vias 0 -> 1
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
Commit message: brd edit
Parts:
- moved C3 0.28 mm to (31.4, 32.7)
- moved C8 0.28 mm to (31.4, 34.8)
Routing:
- net USART3_TX: track 0.00 -> 21.9 mm, vias 0 -> 1
- net USART3_RX: track 0.00 -> 20.8 mm, vias 0 -> 2
- net GND: track 21.0 -> 35.6 mm
- net USART6_TX: track 20.6 -> 25.2 mm
- net USART6_RX: track 19.4 -> 23.2 mm, vias 0 -> 2
- net VDD: track 27.7 -> 26.0 mm
- net I2C2_SCL: track 27.6 -> 26.1 mm, vias 1 -> 0
- net I2C2_SDA: track 26.3 -> 26.0 mm, vias 1 -> 0

Commit message: edit brd
Parts:
- moved C9 0.38 mm to (40.7, 43.6)
- moved U2 0.25 mm to (34.5, 29.6)
- moved R3 0.18 mm to (45.5, 36.1)
- moved C5 0.13 mm to (41.2, 36.2)
Routing:
- net VSSA: track 4.47 -> 8.63 mm
- net USART2_RX: track 16.7 -> 15.5 mm
- net USART6_TX: track 25.2 -> 24.3 mm
- net I2C2_SDA: track 26.0 -> 25.2 mm, vias 0 -> 1
- net GND: track 35.6 -> 36.3 mm
- net VDD: track 26.0 -> 26.5 mm
- net I2C2_SCL: track 26.1 -> 26.0 mm, vias 0 -> 1

Commit message: data upload
Parts:
- removed C12: 4.7uF, Hexabitz:C-0805-POL
- added C10: 100nF, Hexabitz:C-0603
- C11: value 100nf -> 4.7uF; device Hexabitz:C-0603 -> Hexabitz:C-0805-POL
- moved C11 2.22 mm to (26.8, 30.7)
Connections:
- net GND: now also C10.2; no longer C12.2
- net VDD: now also C10.1; no longer C12.1
Routing:
- net VDD: track 26.5 -> 21.9 mm
Other:
- board text added: "H09R90"
- board text removed: "H0BR40"
