File: Design/H09R9x.sch (EAGLE design)
At the start: 25 parts, among them P1 HEXABIT_17.32, U2 TSD305-1C55, X1 XTALL_CSTCE8M00G52

Commit message: first version sch brd .
Parts:
- C2, C4, C7: device Hexabitz:C-0805-POL -> Hexabitz:C-0805
- R1: OCTOPART_URL https://octopart.com/search?q=RC0603FR-07270RL&start=0 -> https://octopart.com/erj-3geyj271v-panasonic-55560546; TOLERANCE 5% -> 1%
- R2: OCTOPART_URL https://octopart.com/rc0603jr-070rl-yageo-1241539?r=sp&s=X2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 -> https://octopart.com/crcw06030000z0eahp-vishay-44320230
- R3: OCTOPART_URL https://octopart.com/search?q=RC0603JR-0710KL&start=0 -> https://octopart.com/crcw060310k0jneb-vishay+dale-46603268
Connections:
- net SCL renamed I2C2_SCL
- net SDA renamed I2C2_SDA
- net USART2_RX renamed USART2_RX*
- net USART2_TX renamed USART2_TX*
- removed net +3V3: C10.1, R57.2, R58.2, U2.VDD
- removed net BLED: U1.PB1
- removed net GLED: U1.PB0
- removed net RLED: U1.PA7
- new net INT: U1.PB2
- net GND: now also U1.PA7, U1.PB0, U1.PB8, U1.PB9
- net VDD: now also C10.1, R57.2, R58.2, U2.VDD
Other:
- note added: "0"
- note added: "H08R6"
- note added: "H08R6_Backend"
- note added: "H08R6_Frontend"
- note added: "Time-of-Flight IR Sensor"
- note removed: "H01R0_Frontend"
- note removed: "H09R9"
- note removed: "H09R9_Frontend"
- note removed: "I2C Pins"
- note removed: "Thermopile Sensor"
- note removed: "VDD=3.3 Volts"
- moved on the sheet: C, C10, D, R57, R58, U2
