File: Design/H09R9x.sch (EAGLE design)
At the start: 24 parts, among them P1 HEXABIT_17.32, U1 STM32F091CBU6, U2 TSD305-1C55, X1 XTALL_CSTCE8M00G52

Commit message: data upload
Parts:
- removed C12: 4.7uF, Hexabitz:C-0805-POL
- added C10: 100nF, Hexabitz:C-0603
- C11: value 100nf -> 4.7uF; device Hexabitz:C-0603 -> Hexabitz:C-0805-POL; CAPACITANCE 10nF -> 4.7uF; MFN AVX -> Panasonic; MPN 0603YC103KAT4A -> 10TPU4R7MSI; OCTOPART_URL https://octopart.com/0603yc103kat4a-avx+interconnect+%2F+el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 -> https://octopart.com/10tpu4r7msi-panasonic-29487748; TOLERANCE 10% -> 20%; VOLTAGE_RATING 16.0 V -> 10.0 V
Connections:
- net GND: now also C10.2, C11.-; no longer C11.2, C12.-
- net VDD: now also C10.1, C11.+; no longer C11.1, C12.+
Changed lines of the file:
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@@
 <part name="GND9" library="supply1" library_urn="urn:adsk.eagle:library:371" deviceset="GND" device=""/>
 <part name="U2" library="HEXABITZ_ICs" library_urn="urn:adsk.eagle:library:20064554" deviceset="TSD305-1C55" device="" package3d_urn="urn:adsk.eagle:package:22912731/1"/>
-<part name="C11" library="Hexabitz" deviceset="C-0603" device="" value="100nf">
-<attribute name="CAPACITANCE" value="10nF"/>
-<attribute name="MFN" value="AVX"/>
-<attribute name="MPN" value="0603YC103KAT4A"/>
-<attribute name="OCTOPART_URL" value="https://octopart.com/0603yc103kat4a-avx+interconnect+%2F+elco-2550362"/>
-<attribute name="TOLERANCE" value="10%"/>
-<attribute name="VOLTAGE_RATING" value="16.0 V"/>
-</part>
-<part name="SUPPLY14" library="supply2" deviceset="VDD" device=""/>
 <part name="SUPPLY15" library="supply2" deviceset="VDD" device=""/>
-<part name="GND10" library="supply1" deviceset="GND" device=""/>
 <part name="GND11" library="supply1" deviceset="GND" device=""/>
-<part name="C12" library="Hexabitz" deviceset="C-0805-POL" device="" value="4.7uF">
+<part name="C11" library="Hexabitz" deviceset="C-0805-POL" device="" value="4.7uF">
 <attribute name="CAPACITANCE" value="4.7uF"/>
 <attribute name="MFN" value="Panasonic"/>
@@
 <part name="SUPPLY16" library="supply2" deviceset="VDD" device=""/>
 <part name="GND12" library="supply1" deviceset="GND" device=""/>
+<part name="C10" library="Hexabitz" deviceset="C-0603" device="" value="100nF">
+<attribute name="CAPACITANCE" value="100nF"/>
+<attribute name="MFN" value="AVX"/>
+<attribute name="MPN" value="0603YC104K4T2A"/>
+<attribute name="OCTOPART_URL" value="https://octopart.com/0603yc104k4t2a-avx+interconnect+%2F+elco-8120651"/>
+<attribute name="TOLERANCE" value="10%"/>
+<attribute name="VOLTAGE_RATING" value="16.0 V"/>
+</part>
+<part name="GND13" library="supply1" deviceset="GND" device=""/>
+<part name="SUPPLY17" library="supply2" deviceset="VDD" device=""/>
 </parts>
 <sheets>
@@
 <attribute name="VALUE" x="170.18" y="73.66" size="1.778" layer="95"/>
 </instance>
-<instance part="C11" gate="G$1" x="130.81" y="85.09" smashed="yes">
-<attribute name="NAME" x="132.334" y="88.011" size="1.778" layer="95"/>
-<attribute name="VALUE" x="132.334" y="82.931" size="1.778" layer="96"/>
-</instance>
-<instance part="SUPPLY14" gate="G$1" x="130.81" y="96.52" smashed="yes">
-<attribute name="VALUE" x="133.985" y="100.965" size="1.778" layer="96" rot="R180"/>
-</instance>
 <instance part="SUPPLY15" gate="G$1" x="135.89" y="96.52" smashed="yes">
 <attribute name="VALUE" x="139.065" y="100.965" size="1.778" layer="96" rot="R180"/>
 </instance>
-<instance part="GND10" gate="1" x="130.81" y="78.74" smashed="yes">
-<attribute name="VALUE" x="128.27" y="76.2" size="1.778" layer="96"/>
-</instance>
 <instance part="GND11" gate="1" x="135.89" y="78.74" smashed="yes">
 <attribute name="VALUE" x="133.35" y="76.2" size="1.778" layer="96"/>
 </instance>
-<instance part="C12" gate="G$1" x="135.89" y="87.63" smashed="yes" rot="MR0">
+<instance part="C11" gate="G$1" x="135.89" y="87.63" smashed="yes" rot="MR0">
 <attribute name="NAME" x="141.224" y="88.265" size="1.778" layer="95" rot="MR0"/>
 <attribute name="VALUE" x="145.034" y="84.709" size="1.778" layer="96" rot="MR0"/>
@@
 <attribute name="VALUE" x="156.21" y="81.28" size="1.778" layer="96" rot="R270"/>
 </instance>
+<instance part="C10" gate="G$1" x="124.46" y="85.09" smashed="yes">
+<attribute name="NAME" x="125.984" y="88.011" size="1.778" layer="95"/>
+<attribute name="VALUE" x="125.984" y="82.931" size="1.778" layer="96"/>
+</instance>
+<instance part="GND13" gate="1" x="124.46" y="80.01" smashed="yes">
+<attribute name="VALUE" x="121.92" y="77.47" size="1.778" layer="96"/>
+</instance>
+<instance part="SUPPLY17" gate="G$1" x="124.46" y="92.71" smashed="yes">
+<attribute name="VALUE" x="127.635" y="97.155" size="1.778" layer="96" rot="R180"/>
+</instance>
 </instances>
 <busses>
@@
 <net name="VDD" class="0">
 <segment>
-<pinref part="C11" gate="G$1" pin="1"/>
-<pinref part="SUPPLY14" gate="G$1" pin="VDD"/>
-<wire x1="130.81" y1="93.98" x2="130.81" y2="90.17" width="0.1524" layer="91"/>
-</segment>
-<segment>
 <pinref part="SUPPLY15" gate="G$1" pin="VDD"/>
 <wire x1="135.89" y1="93.98" x2="135.89" y2="90.17" width="0.1524" layer="91"/>
-<pinref part="C12" gate="G$1" pin="+"/>
+<pinref part="C11" gate="G$1" pin="+"/>
 </segment>
 <segment>
@@
 <wire x1="163.83" y1="93.98" x2="165.1" y2="93.98" width="0.1524" layer="91"/>
 </segment>
-</net>
-<net name="GND" class="0">
 <segment>
-<pinref part="C11" gate="G$1" pin="2"/>
-<pinref part="GND10" gate="1" pin="GND"/>
-<wire x1="130.81" y1="81.28" x2="130.81" y2="82.55" width="0.1524" layer="91"/>
+<pinref part="C10" gate="G$1" pin="1"/>
+<pinref part="SUPPLY17" gate="G$1" pin="VDD"/>
 </segment>
+</net>
+<net name="GND" class="0">
 <segment>
 <pinref part="GND11" gate="1" pin="GND"/>
 <wire x1="135.89" y1="81.28" x2="135.89" y2="82.55" width="0.1524" layer="91"/>
-<pinref part="C12" gate="G$1" pin="-"/>
+<pinref part="C11" gate="G$1" pin="-"/>
 </segment>
 <segment>
@@
 <wire x1="161.29" y1="78.74" x2="165.1" y2="78.74" width="0.1524" layer="91"/>
 </segment>
+<segment>
+<pinref part="C10" gate="G$1" pin="2"/>
+<pinref part="GND13" gate="1" pin="GND"/>
+</segment>
 </net>
